File: SmokESP8266.kicad_pcb (KiCad board)
At the start: 2 copper layers, 57.2 x 61 mm, 32 parts, among them J1 USB_OTG, J2 Cnctor, J3 Sens1Val, J4 Sens1Pwr, J5 ExtraGPIO, K1 SRD-05VDC-SL-C, P1 ProgHeader, Q1 2N3904, SW1 RST, SW2 BOOT, U1 ESP32-WROOM, U2 240x240TFT, U3 AP111733

Commit message: Add files via upload
Parts:
- removed the G*** at (124.5, 93.7)
- removed the G*** at (101.6, 112.8)
- removed P1: ProgHeader, Socket_Strips:Socket_Strip_Straight_1x05_Pitch2.54mm
- removed REF***: CE-Logo_8.5x6mm_SilkScreen, Symbols:CE-Logo_8.5x6mm_SilkScreen
- removed REF***: OSHW-Symbol_6.7x6mm_SilkScreen, Symbols:OSHW-Symbol_6.7x6mm_SilkScreen
- added C7: 10uF, Capacitors_SMD:C_0603_HandSoldering, F.Cu at (87.2, 85.5)
- added C8: 100nF, Capacitors_SMD:C_1206_HandSoldering, B.Cu at (100.1, 75.8)
- added D3: IR-LED, LEDs:LED_D5.0mm_FlatTop, B.Cu at (114.3, 77.0)
- added G***: LOGO, 18650:SOALogo2, B.Cu at (123.7, 115.1)
- added J6: ALIMCapt, Terminal_Blocks:TerminalBlock_bornier-2_P5.08mm, F.Cu at (89.5, 127.9)
- added Q2: S8050, TO_SOT_Packages_SMD:SOT-23, F.Cu at (100.7, 94.4)
- added Q3: S8050, TO_SOT_Packages_SMD:SOT-23, F.Cu at (107.3, 94.4)
- added Q4: BSS138, TO_SOT_Packages_SMD:SOT-23, F.Cu at (93.9, 118.1)
- added Q5: BSS138, TO_SOT_Packages_SMD:SOT-23, F.Cu at (98.4, 118.1)
- added Q6: 2N2222, TO_SOT_Packages_THT:TO-92_Inline_Narrow_Oval, F.Cu at (115.3, 81.5)
- added R10: 10k, Resistors_SMD:R_1206_HandSoldering, F.Cu at (107.9, 114.0)
- added R11: 4.7k, Resistors_SMD:R_1206_HandSoldering, F.Cu at (83.8, 78.1)
- added R12: 470R, Resistors_SMD:R_1206_HandSoldering, B.Cu at (115.1, 73.2)
- added R5: 12k, Resistors_SMD:R_0805_HandSoldering, F.Cu at (87.5, 94.6)
- added R6: 12k, Resistors_SMD:R_0805_HandSoldering, F.Cu at (94.1, 96.6)
- added R7: 10k, Resistors_SMD:R_1206_HandSoldering, F.Cu at (108.0, 117.6)
- added R8: 10k, Resistors_SMD:R_1206_HandSoldering, F.Cu at (107.9, 110.7)
- added R9: 10k, Resistors_SMD:R_1206_HandSoldering, F.Cu at (108.0, 120.7)
- added U4: CP2104, Housings_DFN_QFN:QFN-24-1EP_4x4mm_Pitch0.5mm, F.Cu at (90.6, 103.1)
- added U5: DHT11, 18650:DHT11-debout, F.Cu at (93.2, 74.8)
- moved J3 53.4 mm to (102.1, 127.9), turned to 0 degrees
- moved SW2 23.9 mm to (98.7, 105.5)
- moved SW1 18.3 mm to (83.2, 109.2)
- moved C3 18.2 mm to (108.0, 103.5)
- moved R1 14.2 mm to (100.6, 110.7)
- moved C1 6.01 mm to (93.5, 110.7)
- moved J5 3.69 mm to (103.9, 74.0), turned to 90 degrees
- moved U3 1.53 mm to (107.7, 83.9)
- moved J1 1.02 mm to (81.9, 88.6)
Connections:
- net Net-(C3-Pad1) renamed /RESETB
- net Net-(C4-Pad1) renamed /Bootb
- J1 pad 2: Net-(J1-Pad2) -> /D-
- J1 pad 3: Net-(J1-Pad3) -> /D+
- J1 pad 4: Net-(J1-Pad4) -> (no net)
- J3 pad 1: /GPIO15 -> /5vPM25
- J3 pad 2: /IO21 -> /5vPM1
- U1 pad 10: /IO25 -> (no net)
- U1 pad 12: /IO27 -> (no net)
- U1 pad 14: /Touch5 -> (no net)
- U1 pad 16: /Touch4 -> (no net)
- U1 pad 17: Net-(U1-Pad17) -> (no net)
- U1 pad 18: Net-(U1-Pad18) -> (no net)
- U1 pad 19: Net-(U1-Pad19) -> (no net)
- U1 pad 20: Net-(U1-Pad20) -> (no net)
- U1 pad 21: Net-(U1-Pad21) -> (no net)
- U1 pad 22: Net-(U1-Pad22) -> (no net)
- U1 pad 23: /GPIO15 -> /3vPM25
- U1 pad 24: /Touch3 -> (no net)
- U1 pad 31: /MISO -> (no net)
- U1 pad 32: Net-(U1-Pad32) -> (no net)
- U1 pad 33: /IO21 -> /3vPM1
- U1 pad 34: /RX -> /RXD0
- U1 pad 35: /TX -> /TXD0
- U1 pad 4: /SVP -> (no net)
- U1 pad 5: /SVN -> (no net)
- U1 pad 6: /IO34 -> (no net)
- U1 pad 7: /IO35 -> (no net)
- U1 pad 9: /IO33 -> (no net)
Routing:
- net +3V3: track 161.3 -> 321.7 mm, vias 0 -> 1
- net GND: track 88.4 -> 176.9 mm, vias 9 -> 23
- net +5V: track 73.0 -> 137.4 mm, vias 3 -> 2
- net /3vPM25: track 0.00 -> 60.9 mm
- net /IO21: track 54.7 -> 0.00 mm, vias 3 -> 0
- net /5vPM1: track 0.00 -> 36.3 mm
- net /5vPM25: track 0.00 -> 35.4 mm, vias 0 -> 1
- net /GPIO15: track 35.3 -> 0.00 mm, vias 1 -> 0
- net /TXD0: track 0.00 -> 33.6 mm
- net /RXD0: track 0.00 -> 33.6 mm
- net /IO17: track 73.0 -> 40.5 mm
- net /RTS: track 0.00 -> 28.3 mm, vias 0 -> 3
- net /3vPM1: track 0.00 -> 25.9 mm, vias 0 -> 2
- net /DTR: track 0.00 -> 24.3 mm, vias 0 -> 2
- net /TX: track 23.0 -> 0.00 mm
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Other:
- board text added: "5v"
- board text added: "ESP32/3.3V Smoke Evacuator Dr CADIC Philippe @pwavrobot"
- board text removed: "CTS"
- board text removed: "DTR"
- board text removed: "ESP32/ESP8266/3.3V Smoke Evacuator Dr CADIC Philippe @pwavrobot"
- board text removed: "GPIO"
- board text removed: "GPIO15"
- board text removed: "GPIO21"
- board text removed: "Prototype of PCB to drive the medical laser smokes device."
- board text removed: "RX"
- board text removed: "TX"
