File: SmokESP8266.sch (KiCad schematic (older format))
At the start: 28 parts, among them J1 USB_OTG, J2 Cnctor, J3 Sens1Val, J4 Sens1Pwr, J5 ExtraGPIO, K1 SRD-05VDC-SL-C, P1 ProgHeader, Q1 2N3904, SW1 RST, SW2 BOOT, U1 ESP32-WROOM, U2 240x240TFT, U3 AP111733

Commit message: Add files via upload
Parts:
- removed P1: ProgHeader, Socket_Strips:Socket_Strip_Straight_1x05_Pitch2.54mm, symbol SmokESP8266-rescue:CONN_01X05-WroomMINI2-rescue
- added C7: 10uF, Capacitors_SMD:C_0603_HandSoldering, symbol Device:C_Small
- added C8: 100nF, Capacitors_SMD:C_1206_HandSoldering, symbol SmokESP8266-rescue:C_Small-WroomMINI2-rescue
- added D3: IR-LED, LEDs:LED_D5.0mm_FlatTop, symbol Device:LED_Small
- added J6: ALIMCapt, Terminal_Blocks:TerminalBlock_bornier-2_P5.08mm, symbol Connector:Conn_01x02_Male
- added Q2, Q3: S8050, TO_SOT_Packages_SMD:SOT-23, symbol Transistor_BJT:S8050
- added Q4, Q5: BSS138, TO_SOT_Packages_SMD:SOT-23, symbol Transistor_FET:BSS138
- added Q6: 2N2222, TO_SOT_Packages_THT:TO-92_Inline_Narrow_Oval, symbol Transistor_BJT:PN2222A
- added R10, R7, R8, R9: 10k, Resistors_SMD:R_1206_HandSoldering, symbol SmokESP8266-rescue:R_Small-WroomMINI2-rescue
- added R11: 4.7k, Resistors_SMD:R_1206_HandSoldering, symbol SmokESP8266-rescue:R_Small-WroomMINI2-rescue
- added R12: 470R, Resistors_SMD:R_1206_HandSoldering, symbol Device:R_Small
- added R5, R6: 12k, Resistors_SMD:R_0805_HandSoldering, symbol Device:R_Small
- added U4: CP2104, Housings_DFN_QFN:QFN-24-1EP_4x4mm_Pitch0.5mm, symbol Interface_USB:CP2104
- added U5: DHT11, 18650:DHT11-debout, symbol Sensor:DHT11
Connections:
- net +3V3: now also C7.2, C8.1, D3.2 (A), Q4.1 (G), Q5.1 (G), R11.1, R7.1, R9.1, U4.5 (VIO), U4.6 (VDD), U4.7 (REGIN), U5.1 (VCC)
- net +5V: now also J6.1 (Pin_1), R10.1, R8.1, U4.8 (VBUS)
- net GND: now also C7.1, C8.2, J6.2 (Pin_2), Q6.1 (E), U4.2 (GND), U4.25 (PAD), U5.4 (GND)
- net GPIO4: now also R12.2
- net IO22: now also R11.2, U5.2 (IO)
- net D-: now reaches J1.2 (D-)
- net D-: now also U4.4 (D-)
- net D+: now reaches J1.3 (D+)
- net D+: now also U4.3 (D+)
- net Bootb: now reaches C4.1, SW2.2, U1.25 (IO0)
- net Bootb: now also Q2.3 (C)
- net RESETB: now reaches C3.1, R1.2, SW1.2, U1.3 (EN)
- net RESETB: now also Q3.3 (C)
- net GPIO15 renamed 3vPM25
- net 3vPM25: now also Q4.2 (S), R7.2; no longer J3.1 (Pin_1)
- net IO21 renamed 3vPM1
- net 3vPM1: now also Q5.2 (S), R9.2; no longer J3.2 (Pin_2)
- net RX renamed RXD0
- net RXD0: now also U4.21 (TXD)
- net TX renamed TXD0
- net TXD0: now also U4.20 (RXD)
- new net: Q3.2 (B), R5.2
- new net: Q2.2 (B), R6.2
- new net: Q6.2 (B), R12.1
- new net: D3.1 (K), Q6.3 (C)
- new net 5vPM1: J3.2 (Pin_2), Q5.3 (D), R10.2
- new net 5vPM25: J3.1 (Pin_1), Q4.3 (D), R8.2
- new net DTR: Q2.1 (E), R5.1, U4.23 (DTR)
- new net RTS: Q3.1 (E), R6.1, U4.19 (RTS)
- no-connect marks 9 -> 20
Other:
- note added: "Temperature detection"
- note added: "V converter 1"
- note added: "V converter 2"
- note removed: "CTS"
- note removed: "DTR"
- note removed: "GND"
- note removed: "RX"
- note removed: "TX"
- moved on the sheet: D1, H1, H2, H3, J1, J2, J3, J4, J5, K1, Q1, R2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
